Commit message: Updated commits for package

File: RSE_ws/src/mybot_pkg/urdf/my_bot.urdf.xacro (robot description, xacro)
@@ -39,5 +39,5 @@
       <origin xyz="0 0 0" rpy="0 0 0" />
       <geometry>
-        <box size="1.0 0.6 0.2" />
+        <box size="${base_length} ${base_width} ${base_height}" />
       </geometry>
       <material name="green" />
@@ -46,5 +46,5 @@
       <origin xyz="0 0 0" rpy="0 0 0" />
       <geometry>
-        <box size="1.0 0.6 0.2" />
+        <box size="${base_length} ${base_width} ${base_height}" />
       </geometry>
     </collision>
@@ -52,5 +52,5 @@
       rpy="0 0 0" xyz="0 0 0"
       mass="${base_mass}"
-      x="1.0" y="0.6" z="0.2" />
+      x="${base_length}" y="${base_width}" z="${base_height}" />
   </link>
   <!-- Front steer and rear wheel joints required for ackermann_steering_controller -->
